File: hardware/revA/accelerometer.kicad_sch (KiCad schematic)
At the start: 3 parts, among them U5 MC3419

Commit message: added p/n to drawing sheet
Other:
- title: (none) -> IMU
Changed lines of the file:
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@@
 (kicad_sch (version 20230121) (generator eeschema)
   (paper "A4")
+  (title_block
+    (title "IMU")
+    (rev "A")
+    (comment 1 "CH")
+    (comment 2 "CH")
+    (comment 3 "RD21-7004")
+  )
   (junction (at 86.36 86.36) (diameter 0) (color 0 0 0 0)
   )
